Commit message: Added virtual laser frame to reflect scan data

File: urdf/edubot.urdf (robot description, URDF)
Before this commit: robot edubot, 8 links, 7 joints
Links:
- added link laser
Joints:
- added joint lidar_link_to_laser: type fixed, parent lidar_link, child laser, origin xyz=0 0 0 rpy=0 0 3.14159
